File: ext_sensor.kicad_sch (KiCad schematic)
At the start: 23 parts, among them J12 533980571, J13 533980571, J14 533980571, J15 533980471, J19 533980771, J21 95278-801A10LF, J6 5013310607, J7 532610871, Q1 BSS138G

Commit message: Layout draft
Changed lines of the file:
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@@
 		(on_board yes)
 		(dnp no)
-		(fields_autoplaced yes)
 		(property "Reference" "#PWR075"
 			(at 203.2 120.65 0)
@@
 		)
 		(property "Value" "+3V3"
-			(at 203.2 111.76 0)
+			(at 203.2 112.776 0)
 			(effects
 				(font
@@
 		)
 		(property "Value" "+3V3"
-			(at 225.552 31.242 0)
+			(at 226.06 31.75 0)
 			(effects
 				(font
@@
 		(on_board yes)
 		(dnp no)
-		(fields_autoplaced yes)
 		(property "Reference" "#PWR067"
 			(at 44.45 104.14 0)
@@
 		)
 		(property "Value" "+5V"
-			(at 44.45 95.25 0)
+			(at 44.196 96.266 0)
 			(effects
 				(font
@@
 		(on_board yes)
 		(dnp no)
-		(fields_autoplaced yes)
 		(property "Reference" "#PWR070"
 			(at 120.65 119.38 0)
@@
 		)
 		(property "Value" "+5V"
-			(at 120.65 110.49 0)
+			(at 120.65 112.014 0)
 			(effects
 				(font
@@
 		(on_board yes)
 		(dnp no)
-		(fields_autoplaced yes)
 		(property "Reference" "#PWR079"
 			(at 110.49 156.21 0)
@@
 		)
 		(property "Value" "+3V3"
-			(at 110.49 147.32 0)
+			(at 110.49 148.59 0)
 			(effects
 				(font
@@
 		(on_board yes)
 		(dnp no)
-		(fields_autoplaced yes)
 		(property "Reference" "#PWR036"
 			(at 38.1 54.61 0)
@@
 		)
 		(property "Value" "+5V"
-			(at 38.1 45.72 0)
+			(at 37.592 46.736 0)
 			(effects
 				(font
@@
 		(on_board yes)
 		(dnp no)
-		(fields_autoplaced yes)
 		(property "Reference" "#PWR0137"
 			(at 83.82 179.07 0)
@@
 		)
 		(property "Value" "+3V3"
-			(at 83.82 170.18 0)
+			(at 83.82 170.942 0)
 			(effects
 				(font
@@
 		(on_board yes)
 		(dnp no)
-		(fields_autoplaced yes)
 		(property "Reference" "#PWR030"
 			(at 241.3 41.91 0)
@@
 		)
 		(property "Value" "+5V"
-			(at 241.3 33.02 0)
+			(at 241.3 33.782 0)
 			(effects
 				(font
@@
 		(on_board yes)
 		(dnp no)
-		(fields_autoplaced yes)
 		(property "Reference" "#PWR071"
 			(at 107.95 119.38 0)
@@
 		)
 		(property "Value" "+3V3"
-			(at 107.95 110.49 0)
+			(at 107.95 111.76 0)
 			(effects
 				(font
@@
 		(on_board yes)
 		(dnp no)
-		(fields_autoplaced yes)
 		(property "Reference" "#PWR078"
 			(at 123.19 156.21 0)
@@
 		)
 		(property "Value" "+5V"
-			(at 123.19 147.32 0)
+			(at 123.19 148.336 0)
 			(effects
 				(font
@@
 		(on_board yes)
 		(dnp no)
-		(fields_autoplaced yes)
 		(property "Reference" "#PWR0136"
 			(at 22.86 179.07 0)
@@
 		)
 		(property "Value" "+5V"
-			(at 22.86 170.18 0)
+			(at 22.86 171.196 0)
 			(effects
 				(font
@@
 		(on_board yes)
 		(dnp no)
-		(fields_autoplaced yes)
 		(property "Reference" "#PWR069"
 			(at 33.02 104.14 0)
@@
 		)
 		(property "Value" "+3V3"
-			(at 33.02 95.25 0)
+			(at 32.766 96.52 0)
 			(effects
 				(font
@@
 		(on_board yes)
 		(dnp no)
-		(fields_autoplaced yes)
 		(property "Reference" "#PWR074"
 			(at 215.9 120.65 0)
@@
 		)
 		(property "Value" "+5V"
-			(at 215.9 111.76 0)
+			(at 215.9 112.776 0)
 			(effects
 				(font
