File: int_sensor.kicad_sch (KiCad schematic)
At the start: 36 parts, among them IC1 ADS7828E/2K5, IC2 ADS7828E/2K5, J16 U.FL-R-SMT(01), J3 0787881014, J4 0787881014, J5 0877591014, J8 533980271, Q2 BSS138G, Q3 BSS138G, U6 BME280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

Commit message: Layout draft
Connections:
- net RF_IN_EXT: now reaches C27.1, D9.1 (K), J16.3 (SIG), R16.2
- net I2C_SD renamed I2S_SD
Changed lines of the file:
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@@
 		)
 	)
+	(label "RF_IN_EXT"
+		(at 234.95 133.35 0)
+		(fields_autoplaced yes)
+		(effects
+			(font
+				(size 1.27 1.27)
+			)
+			(justify left bottom)
+		)
+	)
 	(global_label "I2S_WS"
 		(shape input)
@@
 		)
 	)
-	(global_label "I2C_SD"
+	(global_label "I2S_SD"
 		(shape output)
 		(at 158.75 49.53 0)
@@
 		)
 		(property "Intersheetrefs" "${INTERSHEET_REFS}"
-			(at 168.2666 49.53 0)
+			(at 168.2061 49.53 0)
 			(effects
 				(font
@@
 					(unit 1)
 				)
+			)
+		)
+	)
+	(symbol
+		(lib_id "power:PWR_FLAG")
+		(at 243.84 49.53 0)
+		(unit 1)
+		(exclude_from_sim no)
+		(in_bom yes)
+		(on_board yes)
+		(dnp no)
+		(fields_autoplaced yes)
+		(property "Reference" "#FLG011"
+			(at 243.84 47.625 0)
+			(effects
+				(font
+					(size 1.27 1.27)
+				)
+				(hide yes)
+			)
+		)
+		(property "Value" "PWR_FLAG"
+			(at 243.84 44.45 0)
+			(effects
+				(font
+					(size 1.27 1.27)
+				)
+				(hide yes)
+			)
+		)
+		(property "Footprint" ""
+			(at 243.84 49.53 0)
+			(effects
+				(font
+					(size 1.27 1.27)
+				)
+				(hide yes)
+			)
+		)
+		(property "Datasheet" "~"
+			(at 243.84 49.53 0)
+			(effects
+				(font
+					(size 1.27 1.27)
+				)
+				(hide yes)
+			)
+		)
+		(property "Description" "Special symbol for telling ERC where power comes from"
+			(at 243.84 49.53 0)
+			(effects
+				(font
+					(size 1.27 1.27)
+				)
+				(hide yes)
+			)
+		)
+		(pin "1"
+		)
+		(instances
+			(project "airu-base-hardware"
+				(path "/f343fe42-6458-4f46-b8bc-a00e99eb8c9a/dac03172-a2c5-4303-923a-d3dc972d93b4"
+					(reference "#FLG011")
+					(unit 1)
+				)

Commit message: More mfg readiness tweaks; ext power hdr
Parts:
- TP21, TP22, TP23, TP9: now left out of the parts list
Changed lines of the file:
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@@
 	(title_block
 		(title "TELLUS Networked Sensor Solutions, Inc. ")
-		(date "2025-09-16")
+		(date "2025-10-28")
 		(rev "v1.0.0")
 	)
@@
 		(unit 1)
 		(exclude_from_sim no)
-		(in_bom yes)
+		(in_bom no)
 		(on_board yes)
 		(dnp no)
@@
 		(unit 1)
 		(exclude_from_sim no)
-		(in_bom yes)
+		(in_bom no)
 		(on_board yes)
 		(dnp no)
@@
 		(unit 1)
 		(exclude_from_sim no)
-		(in_bom yes)
+		(in_bom no)
 		(on_board yes)
 		(dnp no)
@@
 		(unit 1)
 		(exclude_from_sim no)
-		(in_bom yes)
+		(in_bom no)
 		(on_board yes)
 		(dnp no)
