File: mcu.kicad_sch (KiCad schematic)
At the start: 41 parts, among them J1 12402012E212A, J2 DM3AT-SF-PEJM5, J9 20021121-00006C4LF, SW1 B3F-3100, U1 ESP32-S3-WROOM-1-N8

Commit message: Layout draft
Connections:
- net I2C_SD renamed I2S_SD
Other:
- moved on the sheet: D14, J9

Commit message: More mfg readiness tweaks; ext power hdr
Parts:
- TP10, TP11, TP20: now left out of the parts list
Changed lines of the file:
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@@
 	(title_block
 		(title "TELLUS Networked Sensor Solutions, Inc. ")
-		(date "2025-09-16")
+		(date "2025-10-28")
 		(rev "v1.0.0")
 		(company "TELLUS Networked Sensor Solutions, Inc. ")
@@
 		(unit 1)
 		(exclude_from_sim no)
-		(in_bom yes)
+		(in_bom no)
 		(on_board yes)
 		(dnp no)
@@
 		(unit 1)
 		(exclude_from_sim no)
-		(in_bom yes)
+		(in_bom no)
 		(on_board yes)
 		(dnp no)
@@
 		(unit 1)
 		(exclude_from_sim no)
-		(in_bom yes)
+		(in_bom no)
 		(on_board yes)
 		(dnp no)
