File: network.kicad_sch (KiCad schematic)
At the start: 7 parts, among them J10 NPPN101BFLC-RC, J11 NPPN101BFLC-RC

Commit message: More mfg readiness tweaks; ext power hdr
Parts:
- added J20: 10129380-902001BLF, airu_library:AMPHENOL_10129380-902001BLF, symbol Connector:Conn_01x02_Pin
Connections:
- net +5V_NET_IN: now also J20.1 (Pin_1)
- net GND: now also J20.2 (Pin_2)
Other:
- note added: "External Power Connection"
