File: power.kicad_sch (KiCad schematic)
At the start: 50 parts, among them U10 AP22811AW5-7, U11 TPS72748DSER, U12 MAX40200AUK, U3 TPS2054BDR, U8 LM66200DRLR, U9 AP22811AW5-7

Commit message: Layout draft
Parts:
- removed PS1: TPS62162DSGR, airu_library:SON50P200X200X80-9N, symbol airu_library:TPS62162DSGR
- removed R25: 1.21M, Resistor_SMD:R_0603_1608Metric, symbol Device:R
- removed R26: 383K, Resistor_SMD:R_0603_1608Metric, symbol Device:R
- removed R27: 100K, Resistor_SMD:R_0603_1608Metric, symbol Device:R
- added C69: 100nF, Capacitor_SMD:C_0603_1608Metric, symbol Device:C
- added C70: 22uF, Capacitor_SMD:C_0603_1608Metric, symbol Device:C
- added U13: AP63203WU-7, airu_library:AP63203WU-7_DIO, symbol airu_library:AP63203WU-7
- C52: value 68uF -> 100nF; footprint Capacitor_SMD:C_1206_3216Metric -> Capacitor_SMD:C_0603_1608Metric; Manufacturer_Name TDK Corporation -> YAGEO; Manufacturer_PN C3216X5R1A686M160AC -> CC0603KRX7R7BB104
- L49: value 2.2uH -> 3.9uH; footprint airu_library:IND_VLS3012HBX_TDK -> airu_library:IND_ASPI-0628-3R9M-T1; Manufacturer_Name TDK Corporation -> Bourns; Manufacturer_PN VLS3012HBX-2R2M -> ASPI-0628-3R9M-T
- U8: footprint SOT-5X3_DRL_TEX -> airu_library:SOT-5X3_DRL_TEX
Connections:
- net +3V3_IDLE: now also C70.1, U13.1 (FB)
- net +5V_IDLE: now also U13.2 (EN), U13.3 (VIN)
- net GND: now also C70.2, U13.4 (GND)
- net at L49.2: now also C69.2, U13.5 (SW)
- new net: C69.1, U13.6 (BST)
Other:
- note added: "3.3V Load Switch (Max 2A)"
- note added: "3.3V SMPS (Max 2A)"
- note removed: "3.3V Load Switch (Max 1A)"
- note removed: "3.3V SMPS (Max 1A)"
- moved on the sheet: C50, C51, L49, TP5

Commit message: More mfg readiness tweaks; ext power hdr
Parts:
- TP1, TP5, TP6, TP7, TP8: now left out of the parts list
- U13: Manufacturer_Name (none) -> Diodes Incorporated; Manufacturer_PN (none) -> AP63203WU-7
Changed lines of the file:
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@@
 	(title_block
 		(title "TELLUS Networked Sensor Solutions, Inc. ")
-		(date "2025-09-16")
+		(date "2025-10-28")
 		(rev "v1.0.0")
 	)
@@
 		(unit 1)
 		(exclude_from_sim no)
-		(in_bom yes)
+		(in_bom no)
 		(on_board yes)
 		(dnp no)
@@
 		(unit 1)
 		(exclude_from_sim no)
-		(in_bom yes)
+		(in_bom no)
 		(on_board yes)
 		(dnp no)
@@
 			)
 		)
-		(property "Description" ""
+		(property "Description" "IC, DC-DC BUCK, 3.3V, 2A, TSOT23-6"
+			(at 59.69 106.68 0)
+			(effects
+				(font
+					(size 1.27 1.27)
+				)
+				(hide yes)
+			)
+		)
+		(property "Manufacturer_Name" "Diodes Incorporated"
+			(at 59.69 106.68 0)
+			(effects
+				(font
+					(size 1.27 1.27)
+				)
+				(hide yes)
+			)
+		)
+		(property "Manufacturer_PN" "AP63203WU-7"
 			(at 59.69 106.68 0)
 			(effects
@@
 		(unit 1)
 		(exclude_from_sim no)
-		(in_bom yes)
+		(in_bom no)
 		(on_board yes)
 		(dnp no)
@@
 		(unit 1)
 		(exclude_from_sim no)
-		(in_bom yes)
+		(in_bom no)
 		(on_board yes)
 		(dnp no)
@@
 		(unit 1)
 		(exclude_from_sim no)
-		(in_bom yes)
+		(in_bom no)
 		(on_board yes)
 		(dnp no)

Commit message: Tweaks
Parts:
- L49: Manufacturer_Name Bourns -> Abracon LLC
- U12: Manufacturer_PN MAX40200AUK -> MAX40200AUK+T
Changed lines of the file:
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@@
 			)
 		)
-		(property "Manufacturer_PN" "MAX40200AUK"
+		(property "Manufacturer_PN" "MAX40200AUK+T"
 			(at 80.01 67.31 0)
 			(effects
@@
 			)
 		)
-		(property "Manufacturer_Name" "Bourns"
+		(property "Manufacturer_Name" "Abracon LLC"
 			(at 110.49 109.22 0)
 			(effects
